File: relogger_PCB/RELogger PCB KICAD/RELogger_PCB_v1.sch (KiCad schematic (older format))
At the start: 45 parts, among them K1 ANEMOM1, P1 EXTERNAL PSU, P10 VANE, P11 SERIAL, P12 SOFT_SERIAL, P13 D6_D7, P14 AC_IN, P15 ANEMOM2, P2 BATTERY, P22 A_IN_45, P23 AGND_GND, P3 SOLAR, P4 A_IN_01, P5 A_IN_23, P6 I2C_1, P7 I2C_2, P8 V_EXT, P9 3V3_VREF, SW1 CALIBRATE, SW2 SW_PUSH_SMALL_H, SW4 SW_PUSH_SMALL_H, U1 MCP3208

Commit message: Re load of new PCB
Parts:
- added LOGO2: CONN_1, CuriousElectric3:TCEC_Words_13mm, symbol CONN_1
- HOLE1: footprint (none) -> REInnovationFootprint:3mm_hole_relogger
- LOGO1: footprint (none) -> CuriousElectric3:CEC_Globe_10mm_FCU
- SW1: symbol SPST-RESCUE-RELogger_PCB_v1 -> SPST
- U1: symbol MCP3208-RESCUE-RELogger_PCB_v1 -> MCP3208
Connections:
- net Arduino Uno/D8: now also SW1.2
- net GND: now also SW1.1
- net Hall_to_freq/Vcc_OUT renamed Hall_to_freq/Vss_OUT
- no-connect marks 6 -> 7
Changed lines of the file:
@@
 LIBS:matts_components
 LIBS:linear2
-LIBS:ds3231
-LIBS:micro_sd
 LIBS:RELogger_PCB_v1-cache
 EELAYER 25 0
@@
 F 0 "HOLE1" H 6680 6700 40  0000 L CNN
 F 1 "CONN_1" H 6600 6755 30  0001 C CNN
-F 2 "" H 6600 6700 60  0001 C CNN
+F 2 "REInnovationFootprint:3mm_hole_relogger" H 6600 6700 60  0001 C CNN
 F 3 "" H 6600 6700 60  0001 C CNN
 	1    6600 6700
@@
 $EndComp
 $Comp
-L SPST-RESCUE-RELogger_PCB_v1 SW1
+L SPST SW1
 U 1 1 53A2FA41
 P 7250 2700
@@
 F 0 "LOGO1" H 6680 7150 40  0000 L CNN
 F 1 "CONN_1" H 6600 7205 30  0001 C CNN
-F 2 "" H 6600 7150 60  0001 C CNN
+F 2 "CuriousElectric3:CEC_Globe_10mm_FCU" H 6600 7150 60  0001 C CNN
 F 3 "" H 6600 7150 60  0000 C CNN
 	1    6600 7150
@@
 F0 "Hall_to_freq" 60
 F1 "Hall_to_freq.sch" 60
-F2 "Vcc" I L 9300 5750 60
-F3 "GND" I L 9300 6050 60
-F4 "Freq_Out" O L 9300 5900 60
-F5 "Hall_In" I R 10250 5900 60
-F6 "GND_OUT" O R 10250 6050 60
-F7 "Vcc_OUT" O R 10250 5750 60
+F2 "GND" I L 9300 6050 60
+F3 "Freq_Out" O L 9300 5900 60
+F4 "Hall_In" I R 10250 5900 60
+F5 "GND_OUT" O R 10250 6050 60
+F6 "Vss" I L 9300 5750 60
+F7 "Vss_OUT" O R 10250 5750 60
 $EndSheet
 Wire Wire Line
@@
 	8550 3200 8750 3200
 $Comp
-L MCP3208-RESCUE-RELogger_PCB_v1 U1
+L MCP3208 U1
 U 1 1 58F1890E
 P 6550 4750
@@
 Wire Wire Line
 	10400 4850 10500 4850
+$Comp
+L CONN_1 LOGO2
+U 1 1 58F8AC2F
+P 6600 7300
+F 0 "LOGO2" H 6680 7300 40  0000 L CNN
+F 1 "CONN_1" H 6600 7355 30  0001 C CNN
+F 2 "CuriousElectric3:TCEC_Words_13mm" H 6600 7300 60  0001 C CNN
+F 3 "" H 6600 7300 60  0000 C CNN
+	1    6600 7300
+	1    0    0    -1
+$EndComp
+NoConn ~ 6450 7300
 $EndSCHEMATC

Commit message: BOM uploaded
Parts:
- removed LOGO2: CONN_1, CuriousElectric3:TCEC_Words_13mm, symbol CONN_1
- HOLE1: footprint REInnovationFootprint:3mm_hole_relogger -> (none)
- LOGO1: footprint CuriousElectric3:CEC_Globe_10mm_FCU -> (none)
- SW1: symbol SPST -> SPST-RESCUE-RELogger_PCB_v1
- U1: symbol MCP3208 -> MCP3208-RESCUE-RELogger_PCB_v1
Connections:
- net Arduino Uno/D8: no longer SW1.2
- net GND: no longer SW1.1
- net Hall_to_freq/Vss_OUT renamed Hall_to_freq/Vcc_OUT
- no-connect marks 7 -> 6
Changed lines of the file:
@@
 LIBS:matts_components
 LIBS:linear2
+LIBS:ds3231
+LIBS:micro_sd
 LIBS:RELogger_PCB_v1-cache
 EELAYER 25 0
@@
 F 0 "HOLE1" H 6680 6700 40  0000 L CNN
 F 1 "CONN_1" H 6600 6755 30  0001 C CNN
-F 2 "REInnovationFootprint:3mm_hole_relogger" H 6600 6700 60  0001 C CNN
+F 2 "" H 6600 6700 60  0001 C CNN
 F 3 "" H 6600 6700 60  0001 C CNN
 	1    6600 6700
@@
 $EndComp
 $Comp
-L SPST SW1
+L SPST-RESCUE-RELogger_PCB_v1 SW1
 U 1 1 53A2FA41
 P 7250 2700
@@
 F 0 "LOGO1" H 6680 7150 40  0000 L CNN
 F 1 "CONN_1" H 6600 7205 30  0001 C CNN
-F 2 "CuriousElectric3:CEC_Globe_10mm_FCU" H 6600 7150 60  0001 C CNN
+F 2 "" H 6600 7150 60  0001 C CNN
 F 3 "" H 6600 7150 60  0000 C CNN
 	1    6600 7150
@@
 F0 "Hall_to_freq" 60
 F1 "Hall_to_freq.sch" 60
-F2 "GND" I L 9300 6050 60
-F3 "Freq_Out" O L 9300 5900 60
-F4 "Hall_In" I R 10250 5900 60
-F5 "GND_OUT" O R 10250 6050 60
-F6 "Vss" I L 9300 5750 60
-F7 "Vss_OUT" O R 10250 5750 60
+F2 "Vcc" I L 9300 5750 60
+F3 "GND" I L 9300 6050 60
+F4 "Freq_Out" O L 9300 5900 60
+F5 "Hall_In" I R 10250 5900 60
+F6 "GND_OUT" O R 10250 6050 60
+F7 "Vcc_OUT" O R 10250 5750 60
 $EndSheet
 Wire Wire Line
@@
 	8550 3200 8750 3200
 $Comp
-L MCP3208 U1
+L MCP3208-RESCUE-RELogger_PCB_v1 U1
 U 1 1 58F1890E
 P 6550 4750
@@
 Wire Wire Line
 	10400 4850 10500 4850
-$Comp
-L CONN_1 LOGO2
-U 1 1 58F8AC2F
-P 6600 7300
-F 0 "LOGO2" H 6680 7300 40  0000 L CNN
-F 1 "CONN_1" H 6600 7355 30  0001 C CNN
-F 2 "CuriousElectric3:TCEC_Words_13mm" H 6600 7300 60  0001 C CNN
-F 3 "" H 6600 7300 60  0000 C CNN
-	1    6600 7300
-	1    0    0    -1
-$EndComp
-NoConn ~ 6450 7300
 $EndSCHEMATC
