File: relogger_PCB/RELogger PCB KICAD/RELogger_PCB_v1.sch (KiCad schematic (older format))
At the start: 38 parts, among them K1 ANEMOM1, P1 EXTERNAL PSU, P10 VANE, P11 SERIAL, P12 SOFT_SERIAL, P13 D6_D7, P14 AC_IN, P15 ANEMOM2, P16 CONN_1, P17 CONN_1, P18 CONN_1, P19 CONN_1, P2 BATTERY, P20 CONN_1, P21 CONN_1, P3 SOLAR, P4 A_IN_01, P5 A_IN_23, P6 I2C_1, P7 I2C_2, P8 V_EXT, P9 3V3_VREF, SW1 CALIBRATE

Commit message: Schematic uploaded with Arduino Nano, SD Card connector and DS3231 connector
Parts:
- D1, D2, D3, D4: symbol ZENER -> ZENER-RESCUE-RELogger_PCB_v1
- D5, D6: symbol LED-RESCUE-RELogger_PCB_v1 -> LED-RESCUE-RELogger_PCB_v1-RESCUE-RELogger_PCB_v1
Connections:
- net labels added: MISO, MOSI, SCK, SD_CS
- wire segments 180 -> 173
Changed lines of the file:
@@
 LIBS:matts_components
 LIBS:linear2
+LIBS:ds3231
+LIBS:micro_sd
 LIBS:RELogger_PCB_v1-cache
 EELAYER 25 0
@@
 $EndComp
 $Comp
-L LED-RESCUE-RELogger_PCB_v1 D5
+L LED-RESCUE-RELogger_PCB_v1-RESCUE-RELogger_PCB_v1 D5
 U 1 1 500E6CBF
 P 8000 3850
@@
 F5 "D13" I L 7350 1450 60
 F6 "3V3" I L 7350 1250 60
-F7 "CD" O L 7350 1850 60
-F8 "Vss" I L 7350 2000 60
+F7 "GND" I L 7350 2000 60
 $EndSheet
 $Sheet
@@
 F25 "D8" I R 6500 2250 60
 F26 "D9" I R 6500 2150 60
-F27 "V_USB" O L 5050 2300 60
+F28 "A6" I L 5050 3150 60
+F29 "A7" I L 5050 3250 60
+F30 "5v" I L 5050 2300 60
 $EndSheet
 $Sheet
@@
 F4 "+" I L 1700 6750 60
 F5 "GND" I L 1700 6900 60
-F6 "D2/INT" O R 2500 7000 60
+F6 "D2/SQW" O R 2500 7000 60
 $EndSheet
 $Sheet
@@
 $EndComp
 $Comp
-L LED-RESCUE-RELogger_PCB_v1 D6
+L LED-RESCUE-RELogger_PCB_v1-RESCUE-RELogger_PCB_v1 D6
 U 1 1 54658A3E
 P 8150 800
@@
 $EndComp
 Text HLabel 3450 1400 2    60   Output ~ 0
-Vss
-Text HLabel 7150 2000 0    60   Input ~ 0
 Vss
 Text HLabel 4850 1650 0    60   Input ~ 0
@@
 	1700 6750 1550 6750
 Wire Wire Line
-	6700 1850 7350 1850
-Wire Wire Line
-	6500 2150 6700 2150
-Wire Wire Line
-	6700 2150 6700 1850
-Wire Wire Line
 	7950 800  7850 800
 Wire Wire Line
@@
 	7250 800  7250 1450
 Connection ~ 7250 1450
-Wire Wire Line
-	7150 2000 7350 2000
 Wire Wire Line
 	4450 1750 5050 1750
@@
 	1750 5700 2850 5700
 Connection ~ 2850 5700
-Wire Wire Line
-	2900 1700 3600 1700
-Wire Wire Line
-	3600 1700 3600 2300
-Wire Wire Line
-	3600 2300 5050 2300
 $Comp
 L CONN_4 P5
@@
 Connection ~ 4400 7200
 $Comp
-L ZENER D1
+L ZENER-RESCUE-RELogger_PCB_v1 D1
 U 1 1 57A777BA
 P 3550 3300
@@
 $EndComp
 $Comp
-L ZENER D2
+L ZENER-RESCUE-RELogger_PCB_v1 D2
 U 1 1 57A77978
 P 3850 3300
@@
 $EndComp
 $Comp
-L ZENER D3
+L ZENER-RESCUE-RELogger_PCB_v1 D3
 U 1 1 57A77B3F
 P 4150 3300
@@
 $EndComp
 $Comp
-L ZENER D4
+L ZENER-RESCUE-RELogger_PCB_v1 D4
 U 1 1 57A77CFD
 P 4450 3300
@@
 Text Notes 8350 3600 0    60   ~ 0
 Do all calibration on SD card file?
+Text Label 6500 1750 0    60   ~ 0
+SD_CS
+Text Label 6500 1650 0    60   ~ 0
+MOSI
+Text Label 6500 1550 0    60   ~ 0
+MISO
+Text Label 6500 1450 0    60   ~ 0
+SCK
 $EndSCHEMATC

Commit message: Update of schematic
By ML
Parts:
- removed D5: PWR_3V3, symbol LED-RESCUE-RELogger_PCB_v1-RESCUE-RELogger_PCB_v1
- removed D6: DATA, symbol LED-RESCUE-RELogger_PCB_v1-RESCUE-RELogger_PCB_v1
- removed R6, R7: 1k, symbol R-RESCUE-RELogger_PCB_v1
- added C1: 100n, symbol C
- added D17: WS2811_5mm, symbol WS2811_5mm
- added D5, D6, D7, D8, D9: 5V1, symbol ZENER-RESCUE-RELogger_PCB_v1
- added DISP1: OLED_I2C, symbol OLED_I2C
- added P22: A_IN_45, symbol CONN_4
- added P23: AGND_GND, symbol CONN_01X02
- added SW2, SW4: SW_PUSH_SMALL_H, symbol SW_PUSH_SMALL_H
- added U1: MCP3208, symbol MCP3208
- R2: value 100k -> 47k
Connections:
- net labels added: A4, A5, A6, A7, CLK_ADC, CS_ADC, DIN_ADC, DOUT_ADC, GNDA, IN_ACFREQ, IN_AN1, LED_WS2811, Rx, Rx_SOFT, SW_A, SW_B, Tx, Tx_SOFT, VANE, VBATT, VEXT
- net labels removed: PWR
- wire segments 173 -> 221
- no-connect marks 6 -> 8
Other:
- note removed: "Controlled 3V3 Power\nOnly ON when PWR LOW"
- note removed: "MAX 100mA"
- moved on the sheet: D1, D2, D3, D4, F1, F2, K1, P1, P10, P11, P12, P13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

Commit message: Schematic update and PCB initial run
Parts:
- removed D17: WS2811_5mm, symbol WS2811_5mm
- removed P18, P19, P20: CONN_1, symbol CONN_1
- added D17: WS2811_EpiStar_8mm, REInnovationFootprint:TH_WS2811_LED_8mm, symbol WS2811_EpiStar_8mm
- added EN1: CONN_1, symbol CONN_1
- C1: footprint (none) -> matts_components:C1_wide_lg_pad
- D1, D2, D3, D4, D5, D6, D7, D8, D9: footprint (none) -> REInnovationFootprint:TH_Diode_1
- DISP1: footprint (none) -> REInnovationFootprint:TH_OLED1306
- F1: footprint (none) -> REInnovationFootprint:TH_MC36201_FUSE
- F2: footprint (none) -> REInnovationFootprint:TH_MC36188_FUSE
- K1: footprint (none) -> REInnovationFootprint:SIL-3_screw_terminal
- P1, P10, P14, P15, P8: footprint (none) -> REInnovationFootprint:SIL-2_screw_terminal
- P11, P12, P13, P22, P4, P5, P6, P7: footprint (none) -> matts_components:SIL-4_Grove_SIL
- P2, P3: footprint (none) -> REInnovationFootprint:SIL_2_screw_+_JST_2mm
- P23, P9: footprint (none) -> REInnovationFootprint:SM_2_SLDR_JMP
- R1, R2, R3, R4, R5: footprint (none) -> REInnovationFootprint:TH_Resistor_1
- SW1: footprint (none) -> REInnovationFootprint:SIL-2_large_hole
- SW2, SW4: footprint (none) -> REInnovationFootprint:SW_PUSH_SMALL_lg_pad
- U1: footprint (none) -> REInnovationFootprint:DIP-16__300_ELL
- renumbered P21 to HOLE1, P17 to LOGO1, P16 to PCB1
Connections:
- wire segments 221 -> 224
- no-connect marks 8 -> 6
Other:
- note added: "Hardware"
- note removed: "Bolt Holes"
- moved on the sheet: HOLE1, LOGO1, PCB1

Commit message: Small PCB updates
Parts:
- added LOGO2: CONN_1, CuriousElectric3:TCEC_Words_13mm, symbol CONN_1
- HOLE1: footprint (none) -> REInnovationFootprint:3mm_hole_relogger
- LOGO1: footprint (none) -> CuriousElectric3:CEC_Globe_10mm_FCU
Connections:
- net Hall_to_freq/Vcc_OUT renamed Hall_to_freq/Vss_OUT
- no-connect marks 6 -> 7
Changed lines of the file:
@@
 F 0 "HOLE1" H 6680 6700 40  0000 L CNN
 F 1 "CONN_1" H 6600 6755 30  0001 C CNN
-F 2 "" H 6600 6700 60  0001 C CNN
+F 2 "REInnovationFootprint:3mm_hole_relogger" H 6600 6700 60  0001 C CNN
 F 3 "" H 6600 6700 60  0001 C CNN
 	1    6600 6700
@@
 F 0 "LOGO1" H 6680 7150 40  0000 L CNN
 F 1 "CONN_1" H 6600 7205 30  0001 C CNN
-F 2 "" H 6600 7150 60  0001 C CNN
+F 2 "CuriousElectric3:CEC_Globe_10mm_FCU" H 6600 7150 60  0001 C CNN
 F 3 "" H 6600 7150 60  0000 C CNN
 	1    6600 7150
@@
 F0 "Hall_to_freq" 60
 F1 "Hall_to_freq.sch" 60
-F2 "Vcc" I L 9300 5750 60
-F3 "GND" I L 9300 6050 60
-F4 "Freq_Out" O L 9300 5900 60
-F5 "Hall_In" I R 10250 5900 60
-F6 "GND_OUT" O R 10250 6050 60
-F7 "Vcc_OUT" O R 10250 5750 60
+F2 "GND" I L 9300 6050 60
+F3 "Freq_Out" O L 9300 5900 60
+F4 "Hall_In" I R 10250 5900 60
+F5 "GND_OUT" O R 10250 6050 60
+F6 "Vss" I L 9300 5750 60
+F7 "Vss_OUT" O R 10250 5750 60
 $EndSheet
 Wire Wire Line
@@
 Wire Wire Line
 	10400 4850 10500 4850
+$Comp
+L CONN_1 LOGO2
+U 1 1 58F8AC2F
+P 6600 7300
+F 0 "LOGO2" H 6680 7300 40  0000 L CNN
+F 1 "CONN_1" H 6600 7355 30  0001 C CNN
+F 2 "CuriousElectric3:TCEC_Words_13mm" H 6600 7300 60  0001 C CNN
+F 3 "" H 6600 7300 60  0000 C CNN
+	1    6600 7300
+	1    0    0    -1
+$EndComp
+NoConn ~ 6450 7300
 $EndSCHEMATC

Commit message: BOM updated
Parts:
- F1: Description (none) -> Resettable fuse. 0.5A; Supplier 1 (none) -> RS; Supplier 1 Cost (none) -> 0.27; Supplier 1 Part No (none) -> 517-6635
- F2: Description (none) -> Resettable fuse. 0.1A; Supplier 1 (none) -> RS; Supplier 1 Cost (none) -> 0.363; Supplier 1 Part No (none) -> 869-7416
Changed lines of the file:
@@
 F 2 "REInnovationFootprint:TH_MC36188_FUSE" H 1400 4400 50  0001 C CNN
 F 3 "" H 1400 4400 50  0000 C CNN
+F 4 "~" H 1400 4400 60  0000 C CNN "Notes"
+F 5 "Resettable fuse. 0.1A" H 1400 4400 60  0001 C CNN "Description"
+F 6 "~" H 1400 4400 60  0001 C CNN "Manufacturer"
+F 7 "~" H 1400 4400 60  0001 C CNN "Manufacturer Part No"
+F 8 "RS" H 1400 4400 60  0001 C CNN "Supplier 1"
+F 9 "869-7416" H 1400 4400 60  0001 C CNN "Supplier 1 Part No"
+F 10 "0.363" H 1400 4400 60  0001 C CNN "Supplier 1 Cost"
+F 11 "~" H 1400 4400 60  0001 C CNN "Supplier 2"
+F 12 "~" H 1400 4400 60  0001 C CNN "Supplier 2 Part No"
+F 13 "~" H 1400 4400 60  0001 C CNN "Supplier 2 Cost"
 	1    1400 4400
 	1    0    0    -1
@@
 F 2 "REInnovationFootprint:TH_MC36201_FUSE" H 1450 1750 50  0001 C CNN
 F 3 "" H 1450 1750 50  0000 C CNN
+F 4 "~" H 1450 1750 60  0000 C CNN "Notes"
+F 5 "Resettable fuse. 0.5A" H 1450 1750 60  0001 C CNN "Description"
+F 6 "~" H 1450 1750 60  0001 C CNN "Manufacturer"
+F 7 "~" H 1450 1750 60  0001 C CNN "Manufacturer Part No"
+F 8 "RS" H 1450 1750 60  0001 C CNN "Supplier 1"
+F 9 "517-6635" H 1450 1750 60  0001 C CNN "Supplier 1 Part No"
+F 10 "0.27" H 1450 1750 60  0001 C CNN "Supplier 1 Cost"
+F 11 "~" H 1450 1750 60  0001 C CNN "Supplier 2"
+F 12 "~" H 1450 1750 60  0001 C CNN "Supplier 2 Part No"
+F 13 "~" H 1450 1750 60  0001 C CNN "Supplier 2 Cost"
 	1    1450 1750
 	1    0    0    -1

Commit message: update of PCB
Changed lines of the file:
@@
 $EndComp
 NoConn ~ 6450 7300
+$Comp
+L GND-RESCUE-RELogger_PCB_v1 #PWR?
+U 1 1 59306D13
+P 6800 1850
+F 0 "#PWR?" H 6800 1850 30  0001 C CNN
+F 1 "GND" H 6800 1780 30  0001 C CNN
+F 2 "" H 6800 1850 60  0001 C CNN
+F 3 "" H 6800 1850 60  0001 C CNN
+	1    6800 1850
+	1    0    0    -1
+$EndComp
+Wire Wire Line
+	6900 1800 6800 1800
+Wire Wire Line
+	6800 1800 6800 1850
 $EndSCHEMATC

Commit message: Updated schmatic
Debounce switches. Power control for all.
Parts:
- removed DISP1: OLED_I2C, REInnovationFootprint:TH_OLED1306, symbol OLED_I2C
- removed P7: I2C_2, matts_components:SIL-4_Grove_SIL, symbol CONN_4
- removed SW2, SW4: SW_PUSH_SMALL_H, REInnovationFootprint:SW_PUSH_SMALL_lg_pad, symbol SW_PUSH_SMALL_H
- added C2: C, symbol C
- added D19: D_Schottky, symbol D_Schottky
- added P7: AN_JMP, REInnovationFootprint:SIL-2_screw_terminal, symbol CONN_01X02
- added Q1: Q_PMOS_DGS, symbol Q_PMOS_DGS
- added Q3: Q_NPN_CBE, symbol Q_NPN_CBE
- added R7, R9: 100k, symbol R
- added R8: 330, symbol R
- U1: symbol MCP3208 -> MCP3208-RESCUE-RELogger_PCB_v1
- renumbered K1 to P16
Connections:
- net Arduino Uno/5v: now also D19.1 (K)
- net GND: now also Q3.3 (E), R9.2; no longer P12.4 (P4)
- net GNDA: now also C2.2
- net IN_ACFREQ: now also P7.2 (P2); no longer P15.1 (P1)
- net VEXT: now also C2.1
- net Vss: now also D19.2 (A), Q1.1 (D), R7.1; no longer P22.3 (P3), P4.3 (P3), P5.3 (P3)
- new net: P22.3 (P3), P4.3 (P3), P5.3 (P3), Q1.3 (S)
- new net: P12.4 (P4), Q3.1 (C)
- new net: Q3.2 (B), R8.2, R9.1
- new net Hall_to_freq/Freq_IN: P15.1 (P1)
- new net Hall_to_freq/Freq_OUT2: P7.1 (P1)
- new net PWR_EXTI: Q1.2 (G), R7.2
- new net PWR_GPS: R8.1
- no-connect marks 7 -> 6
Other:
- note added: "Power Control\nIn +VE Path"
- note added: "With power control\nIn -ve Path"
- moved on the sheet: D17, D4, D5, D6, D7, D8, D9, EN1, HOLE1, LOGO1, LOGO2, P11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

Commit message: Small updates
Parts:
- added P17: HC12, symbol CONN_01X05
Connections:
- net +3.3V: now also P17.5 (P5)
- net GND: now also P17.4 (P4)
- net Rx_SOFT: now also P17.2 (P2)
- net Tx_SOFT: now also P17.3 (P3)
- new net HC12_SET: P17.1 (P1)
Changed lines of the file:
@@
 	4250 1850 4250 2100
 Connection ~ 4250 2100
+$Comp
+L CONN_01X05 P17
+U 1 1 595D28A0
+P 10650 3450
+F 0 "P17" H 10650 3750 50  0000 C CNN
+F 1 "HC12" V 10750 3450 50  0000 C CNN
+F 2 "" H 10650 3450 50  0000 C CNN
+F 3 "" H 10650 3450 50  0000 C CNN
+F 4 "~" H 10650 3450 60  0001 C CNN "Description"
+F 5 "~" H 10650 3450 60  0001 C CNN "Notes"
+F 6 "~" H 10650 3450 60  0001 C CNN "Manufacturer"
+F 7 "~" H 10650 3450 60  0001 C CNN "Manufacturer Part No"
+F 8 "~" H 10650 3450 60  0001 C CNN "Supplier 1"
+F 9 "~" H 10650 3450 60  0001 C CNN "Supplier 1 Part No"
+F 10 "~" H 10650 3450 60  0001 C CNN "Supplier 2"
+F 11 "~" H 10650 3450 60  0001 C CNN "Supplier 2 Part No"
+F 12 "~" H 10650 3450 60  0001 C CNN "Cost"
+	1    10650 3450
+	1    0    0    1
+$EndComp
+Text HLabel 6300 2250 2    60   Output ~ 0
+HC12_SET
+Wire Wire Line
+	6300 2250 6050 2250
+Text HLabel 10100 3650 0    60   Input ~ 0
+HC12_SET
+Text HLabel 10100 3550 0    60   Input ~ 0
+Rx_SOFT
+Text HLabel 10100 3450 0    60   Input ~ 0
+Tx_SOFT
+$Comp
+L GND-RESCUE-RELogger_PCB_v1 #PWR033
+U 1 1 595D4108
+P 9800 3300
+F 0 "#PWR033" H 9800 3300 30  0001 C CNN
+F 1 "GND" H 9800 3230 30  0001 C CNN
+F 2 "" H 9800 3300 60  0001 C CNN
+F 3 "" H 9800 3300 60  0001 C CNN
+	1    9800 3300
+	1    0    0    -1
+$EndComp
+$Comp
+L +3.3V-RESCUE-RELogger_PCB_v1 #PWR034
+U 1 1 595D4BF6
+P 10150 3200
+F 0 "#PWR034" H 10150 3160 30  0001 C CNN
+F 1 "+3.3V" H 10150 3310 30  0000 C CNN
+F 2 "" H 10150 3200 60  0000 C CNN
+F 3 "" H 10150 3200 60  0000 C CNN
+	1    10150 3200
+	1    0    0    -1
+$EndComp
+Wire Wire Line
+	10450 3250 10150 3250
+Wire Wire Line
+	10150 3250 10150 3200
+Wire Wire Line
+	9800 3300 9800 3200
+Wire Wire Line
+	9800 3200 10000 3200
+Wire Wire Line
+	10000 3200 10000 3350
+Wire Wire Line
+	10000 3350 10450 3350
+Wire Wire Line
+	10100 3450 10450 3450
+Wire Wire Line
+	10100 3550 10450 3550
+Wire Wire Line
+	10100 3650 10450 3650
 $EndSCHEMATC
