File: relogger_PCB/RELogger PCB KICAD/ArduinoUno.sch (KiCad schematic (older format))
At the start: 14 parts, among them IC1 ATMEGA328P-A, P22 FTDI, P23 SERIAL, P24 ISP, SW2 RESET, X1 16MHz

Commit message: Schematic uploaded with Arduino Nano, SD Card connector and DS3231 connector
Parts:
- removed C1: 100uF, symbol CP1-RESCUE-RELogger_PCB_v1
- removed C2, C3: 100nF, symbol C-RESCUE-RELogger_PCB_v1
- removed C4, C5: 22pF, symbol C-RESCUE-RELogger_PCB_v1
- removed D7, D8: D_Schottky, symbol D_Schottky
- removed IC1: ATMEGA328P-A, TQFP32, symbol ATMEGA328P-A-RESCUE-RELogger_PCB_v1
- removed P22: FTDI, symbol CONN_6
- removed P23: SERIAL, symbol CONN_6
- removed P24: ISP, symbol CONN_3X2
- removed R9: 10k, symbol R-RESCUE-RELogger_PCB_v1
- removed SW2: RESET, symbol SPST
- removed X1: 16MHz, symbol CRYSTAL_Matt
- added J2: Arduino_Nano_Header, symbol Arduino_Nano_Header
Connections:
- net labels added: 5v, A6, A7
- net labels removed: V_USB, a0, a1, a2, a3, a4, a5, d0, d1, d10, d11, d12, d13, d2, d3, d4, d5, d6, d7, d8, d9
- wire segments 84 -> 30
- no-connect marks 2 -> 0
Other:
- note removed: "1: 3.3V\n2: RST\n3: Vcc\n4: TxD\n5: RxD\n6: GND"
- note removed: "1: RTS#\n2: Rx\n3: Tx\n4: Vcc\n5: CTS#\n6: GND"
- note removed: "ISP"
- note removed: "OUTPUT FOR SERIAL/USB"
- note removed: "USE 'Off the shelf' Board here?\nWith Serial built in for easy upload?\nPro Micro 3.3V/5V £3.88 (single)\n"

Commit message: Schematic update and PCB initial run
Parts:
- J2: footprint (none) -> REInnovationFootprint:NANO_DIP_30_600
Changed lines of the file:
@@
 F 0 "J2" H 5750 4000 60  0000 C CNN
 F 1 "Arduino_Nano_Header" H 5750 2400 60  0000 C CNN
-F 2 "" H 5750 3200 60  0000 C CNN
+F 2 "REInnovationFootprint:NANO_DIP_30_600" H 5750 3200 60  0001 C CNN
 F 3 "" H 5750 3200 60  0000 C CNN
 	1    5750 3200
