File: relogger_PCB/RELogger PCB KICAD/SolarCharger.sch (KiCad schematic (older format))
At the start: 22 parts, among them Q1 Q_PMOS_GDS, Q2 Q_PMOS_GDS, SW3 ON/OFF, U3 LM2574, U4 MCP1703, U5 MCP73832

Commit message: Schematic uploaded with Arduino Nano, SD Card connector and DS3231 connector
Parts:
- D13: symbol LED -> LED-RESCUE-RELogger_PCB_v1-RESCUE-RELogger_PCB_v1
Changed lines of the file:
@@
 LIBS:matts_components
 LIBS:linear2
+LIBS:ds3231
+LIBS:micro_sd
 LIBS:RELogger_PCB_v1-cache
 EELAYER 25 0
@@
 	8600 2450 8600 2350
 $Comp
-L LED D13
+L LED-RESCUE-RELogger_PCB_v1-RESCUE-RELogger_PCB_v1 D13
 U 1 1 57A0C9C8
 P 6050 4750
+AR Path="/57A0C9C8" Ref="D13"  Part="1"
+AR Path="/546244C7/57A0C9C8" Ref="D13"  Part="1"
 F 0 "D13" H 6050 4850 50  0000 C CNN
 F 1 "LED" H 6050 4650 50  0000 C CNN

Commit message: Update of schematic
By ML
Parts:
- removed Q1: Q_PMOS_GDS, symbol Q_PMOS_GDS
- removed R15: 100k, symbol R
- added D18: D_Schottky, symbol D_Schottky
- Q2: value Q_PMOS_GDS -> RFU9110PBF; Description (none) -> 3.1A P FET; Manufacturer (none) -> Vishay; Manufacturer Part No (none) -> RFU9110PBF; Supplier 1 (none) -> RS; Supplier 1 Cost (none) -> 0.24; Supplier 1 Part No (none) -> 541-1663
- U4: value MCP1703 -> MCP1826S; Description (none) -> 1A LDO low Iq; Manufacturer (none) -> Microchip; Manufacturer Part No (none) -> MCP1826S-3302E/AB; Supplier 1 (none) -> RS; Supplier 1 Cost (none) -> 0.76; Supplier 1 Part No (none) -> 669-5174
- U5: Description (none) -> 500mA Linear Charge control IC; Manufacturer (none) -> Microchip; Manufacturer Part No (none) -> MCP73832T-2DCI/OT; Supplier 1 (none) -> RS; Supplier 1 Cost (none) -> 0.446; Supplier 1 Part No (none) -> 738-6629
Connections:
- net labels removed: PWR_CTRL
- wire segments 64 -> 59
Other:
- note removed: "Power Control"
- moved on the sheet: C11, C13
Changed lines of the file:
@@
 LIBS:matts_components
 LIBS:linear2
-LIBS:ds3231
-LIBS:micro_sd
 LIBS:RELogger_PCB_v1-cache
 EELAYER 25 0
@@
 Comment4 ""
 $EndDescr
-Connection ~ 6100 6450
-Wire Wire Line
-	4750 6850 6100 6850
-Connection ~ 4750 6450
+Connection ~ 10200 5050
+Wire Wire Line
+	8850 5450 10200 5450
+Connection ~ 8850 5050
 $Comp
 L CP1-RESCUE-RELogger_PCB_v1 C13
 U 1 1 5463B713
-P 6100 6650
-F 0 "C13" H 6150 6750 50  0000 L CNN
-F 1 "10uF" H 6150 6550 50  0000 L CNN
-F 2 "" H 6100 6650 60  0001 C CNN
-F 3 "" H 6100 6650 60  0001 C CNN
-	1    6100 6650
+P 10200 5250
+F 0 "C13" H 10250 5350 50  0000 L CNN
+F 1 "10uF" H 10250 5150 50  0000 L CNN
+F 2 "" H 10200 5250 60  0001 C CNN
+F 3 "" H 10200 5250 60  0001 C CNN
+	1    10200 5250
 	1    0    0    -1
 $EndComp
@@
 L CP1-RESCUE-RELogger_PCB_v1 C11
 U 1 1 5463B719
-P 4750 6650
-F 0 "C11" H 4800 6750 50  0000 L CNN
-F 1 "10uF" H 4800 6550 50  0000 L CNN
-F 2 "" H 4750 6650 60  0001 C CNN
-F 3 "" H 4750 6650 60  0001 C CNN
-	1    4750 6650
-	1    0    0    -1
-$EndComp
-Text HLabel 6400 6450 2    60   Output ~ 0
+P 8850 5250
+F 0 "C11" H 8900 5350 50  0000 L CNN
+F 1 "10uF" H 8900 5150 50  0000 L CNN
+F 2 "" H 8850 5250 60  0001 C CNN
+F 3 "" H 8850 5250 60  0001 C CNN
+	1    8850 5250
+	1    0    0    -1
+$EndComp
+Text HLabel 10500 5050 2    60   Output ~ 0
 3V3
 Text HLabel 4150 2700 0    60   Input ~ 0
@@
 L MCP1703-Matt U4
 U 1 1 5467B677
-P 5450 6500
-F 0 "U4" H 5600 6304 60  0000 C CNN
-F 1 "MCP1703" H 5450 6700 60  0000 C CNN
-F 2 "~" H 5450 6500 60  0000 C CNN
-F 3 "~" H 5450 6500 60  0000 C CNN
-	1    5450 6500
+P 9550 5100
+F 0 "U4" H 9700 4904 60  0000 C CNN
+F 1 "MCP1826S" H 9550 5300 60  0000 C CNN
+F 2 "~" H 9550 5100 60  0000 C CNN
+F 3 "http://docs-europe.electrocomponents.com/webdocs/137e/0900766b8137eda2.pdf" H 9550 5100 60  0001 C CNN
+F 4 "~" H 9550 5100 60  0000 C CNN "Notes"
+F 5 "1A LDO low Iq" H 9550 5100 60  0001 C CNN "Description"
+F 6 "Microchip" H 9550 5100 60  0001 C CNN "Manufacturer"
+F 7 "MCP1826S-3302E/AB" H 9550 5100 60  0001 C CNN "Manufacturer Part No"
+F 8 "RS" H 9550 5100 60  0001 C CNN "Supplier 1"
+F 9 "669-5174" H 9550 5100 60  0001 C CNN "Supplier 1 Part No"
+F 10 "0.76" H 9550 5100 60  0001 C CNN "Supplier 1 Cost"
+F 11 "~" H 9550 5100 60  0001 C CNN "Supplier 2"
+F 12 "~" H 9550 5100 60  0001 C CNN "Supplier 2 Part No"
+F 13 "~" H 9550 5100 60  0001 C CNN "Supplier 2 Cost"
+	1    9550 5100
 	1    0    0    -1
 $EndComp
@@
 BATT+
 Wire Wire Line
-	5850 6450 6400 6450
-Wire Wire Line
-	3750 6450 5050 6450
+	9950 5050 10500 5050
 Text HLabel 1750 1000 0    60   Input ~ 0
 EXTERNAL+
@@
 Connection ~ 4150 1850
 Wire Wire Line
-	5450 6750 5450 6850
-Connection ~ 5450 6850
-Text HLabel 5100 7050 0    60   Input ~ 0
-GND
-Wire Wire Line
-	5100 7050 5250 7050
-Wire Wire Line
-	5250 7050 5250 6850
-Connection ~ 5250 6850
+	9550 5350 9550 5450
+Connection ~ 9550 5450
+Text HLabel 9200 5650 0    60   Input ~ 0
+GND
+Wire Wire Line
+	9200 5650 9350 5650
+Wire Wire Line
+	9350 5650 9350 5450
+Connection ~ 9350 5450
 Connection ~ 2000 1850
 $Comp
@@
 F 1 "MCP73832" H 5400 5550 60  0000 C CNN
 F 2 "" H 5500 4700 60  0000 C CNN
-F 3 "" H 5500 4700 60  0000 C CNN
+F 3 "http://ww1.microchip.com/downloads/en/DeviceDoc/20001984g.pdf" H 5500 4700 60  0001 C CNN
+F 4 "~" H 5500 4700 60  0000 C CNN "Notes"
+F 5 "500mA Linear Charge control IC" H 5500 4700 60  0001 C CNN "Description"
+F 6 "Microchip" H 5500 4700 60  0001 C CNN "Manufacturer"
+F 7 "MCP73832T-2DCI/OT" H 5500 4700 60  0001 C CNN "Manufacturer Part No"
+F 8 "RS" H 5500 4700 60  0001 C CNN "Supplier 1"
+F 9 "738-6629" H 5500 4700 60  0001 C CNN "Supplier 1 Part No"
+F 10 "0.446" H 5500 4700 60  0001 C CNN "Supplier 1 Cost"
+F 11 "~" H 5500 4700 60  0001 C CNN "Supplier 2"
+F 12 "~" H 5500 4700 60  0001 C CNN "Supplier 2 Part No"
+F 13 "~" H 5500 4700 60  0001 C CNN "Supplier 2 Cost"
 	1    5500 4700
 	1    0    0    -1
@@
 P 9150 2550
 F 0 "Q2" H 9450 2600 50  0000 R CNN
-F 1 "Q_PMOS_GDS" H 9800 2500 50  0000 R CNN
+F 1 "RFU9110PBF" H 9800 2500 50  0000 R CNN
 F 2 "" H 9350 2650 50  0000 C CNN
-F 3 "" H 9150 2550 50  0000 C CNN
+F 3 "http://docs-europe.electrocomponents.com/webdocs/0791/0900766b807912ad.pdf" H 9150 2550 50  0001 C CNN
+F 4 "~" H 9150 2550 60  0000 C CNN "Notes"
+F 5 "3.1A P FET" H 9150 2550 60  0001 C CNN "Description"
+F 6 "Vishay" H 9150 2550 60  0001 C CNN "Manufacturer"
+F 7 "RFU9110PBF" H 9150 2550 60  0001 C CNN "Manufacturer Part No"
+F 8 "RS" H 9150 2550 60  0001 C CNN "Supplier 1"
+F 9 "541-1663" H 9150 2550 60  0001 C CNN "Supplier 1 Part No"
+F 10 "0.24" H 9150 2550 60  0001 C CNN "Supplier 1 Cost"
+F 11 "~" H 9150 2550 60  0001 C CNN "Supplier 2"
+F 12 "~" H 9150 2550 60  0001 C CNN "Supplier 2 Part No"
+F 13 "~" H 9150 2550 60  0001 C CNN "Supplier 2 Cost"
 	1    9150 2550
 	0    -1   1    0
@@
 Text HLabel 4750 4300 0    60   Input ~ 0
 GND
-Text HLabel 3550 5750 0    60   Input ~ 0
+Text HLabel 8150 5050 0    60   Input ~ 0
 Vss
 Text HLabel 4500 5150 0    60   Input ~ 0
@@
 Text HLabel 4100 3050 0    60   Input ~ 0
 V_USB
-Wire Wire Line
-	4100 3050 7200 3050
 Connection ~ 7200 3050
 $Comp
@@
 	10550 2650 10550 2850
 $Comp
-L Q_PMOS_GDS Q1
-U 1 1 57B9A111
-P 3650 6150
-F 0 "Q1" H 3950 6200 50  0000 R CNN
-F 1 "Q_PMOS_GDS" H 4300 6100 50  0000 R CNN
-F 2 "" H 3850 6250 50  0000 C CNN
-F 3 "" H 3650 6150 50  0000 C CNN
-	1    3650 6150
-	1    0    0    1
-$EndComp
-$Comp
-L R R15
-U 1 1 57B9A118
-P 3350 6400
-F 0 "R15" V 3430 6400 50  0000 C CNN
-F 1 "100k" V 3350 6400 50  0000 C CNN
-F 2 "" V 3280 6400 50  0000 C CNN
-F 3 "" H 3350 6400 50  0000 C CNN
-	1    3350 6400
-	1    0    0    -1
-$EndComp
-Text Notes 3550 6600 0    60   ~ 0
-Power Control
-Wire Wire Line
-	3750 5750 3750 5950
-Wire Wire Line
-	3750 6350 3750 6450
-$Comp
-L GND-RESCUE-RELogger_PCB_v1 #PWR026
-U 1 1 57B9A129
-P 3350 6600
-F 0 "#PWR026" H 3350 6600 30  0001 C CNN
-F 1 "GND" H 3350 6530 30  0001 C CNN
-F 2 "" H 3350 6600 60  0001 C CNN
-F 3 "" H 3350 6600 60  0001 C CNN
-	1    3350 6600
-	1    0    0    -1
-$EndComp
-Wire Wire Line
-	3350 6600 3350 6550
-Wire Wire Line
-	3250 6150 3450 6150
-Wire Wire Line
-	3350 6150 3350 6250
-Text HLabel 3250 6150 0    60   Input ~ 0
-PWR_CTRL
-Connection ~ 3350 6150
-Wire Wire Line
-	3550 5750 3750 5750
+L D_Schottky D18
+U 1 1 58F5FCFA
+P 6050 3050
+F 0 "D18" H 6050 3150 50  0000 C CNN
+F 1 "D_Schottky" H 6050 2950 50  0000 C CNN
+F 2 "" H 6050 3050 50  0000 C CNN
+F 3 "" H 6050 3050 50  0000 C CNN
+	1    6050 3050
+	-1   0    0    1
+$EndComp
+Wire Wire Line
+	4100 3050 5900 3050
+Wire Wire Line
+	6200 3050 7200 3050
+Wire Wire Line
+	8150 5050 9150 5050
 $EndSCHEMATC

Commit message: Schematic update and PCB initial run
Parts:
- removed U4: MCP1826S, ~, symbol MCP1703-Matt
- added U2: MCP1826S, REInnovationFootprint:TO220_MCP1826S, symbol MCP1826S
- C10, C11, C12, C13, C14, C9: footprint (none) -> REInnovationFootprint:C_1V7_TH
- D10, D11, D12, D14, D18: footprint (none) -> REInnovationFootprint:TH_Diode_1
- D13: value LED -> CHRG; footprint (none) -> REInnovationFootprint:TH_LED-5MM_larg_pad
- L1: footprint (none) -> REInnovationFootprint:TH_Inductor
- Q2: footprint (none) -> REInnovationFootprint:TO220_P_FET
- R16, R17, R18: footprint (none) -> REInnovationFootprint:TH_Resistor_1
- SW3: footprint (none) -> matts_components:SW_SPDT_rapid_760271
- U3: footprint (none) -> REInnovationFootprint:DIP-8_300_ELL; Description (none) -> 0.5A step down DC-DC; Manufacturer (none) -> TI; Manufacturer Part No (none) -> LM2574; Supplier 1 (none) -> RS
- U5: footprint (none) -> REInnovationFootprint:SM_SOT-23-5
Changed lines of the file:
@@
 F 0 "C13" H 10250 5350 50  0000 L CNN
 F 1 "10uF" H 10250 5150 50  0000 L CNN
-F 2 "" H 10200 5250 60  0001 C CNN
+F 2 "REInnovationFootprint:C_1V7_TH" H 10200 5250 60  0001 C CNN
 F 3 "" H 10200 5250 60  0001 C CNN
 	1    10200 5250
@@
 F 0 "C11" H 8900 5350 50  0000 L CNN
 F 1 "10uF" H 8900 5150 50  0000 L CNN
-F 2 "" H 8850 5250 60  0001 C CNN
+F 2 "REInnovationFootprint:C_1V7_TH" H 8850 5250 60  0001 C CNN
 F 3 "" H 8850 5250 60  0001 C CNN
 	1    8850 5250
@@
 F 0 "R17" V 6430 4150 50  0000 C CNN
 F 1 "2k" V 6350 4150 50  0000 C CNN
-F 2 "" H 6350 4150 60  0000 C CNN
+F 2 "REInnovationFootprint:TH_Resistor_1" H 6350 4150 60  0001 C CNN
 F 3 "" H 6350 4150 60  0000 C CNN
 	1    6350 4150
@@
 F 0 "R16" V 6130 5250 50  0000 C CNN
 F 1 "470" V 6050 5250 50  0000 C CNN
-F 2 "" H 6050 5250 60  0000 C CNN
+F 2 "REInnovationFootprint:TH_Resistor_1" H 6050 5250 60  0001 C CNN
 F 3 "" H 6050 5250 60  0000 C CNN
 	1    6050 5250
@@
 F 0 "C10" H 4700 4900 50  0000 L CNN
 F 1 "4.7uf" H 4700 4700 50  0000 L CNN
-F 2 "" H 4650 4800 60  0000 C CNN
+F 2 "REInnovationFootprint:C_1V7_TH" H 4650 4800 60  0001 C CNN
 F 3 "" H 4650 4800 60  0000 C CNN
 	1    4650 4800
@@
 F 0 "C14" H 6750 4900 50  0000 L CNN
 F 1 "4.7uf" H 6750 4700 50  0000 L CNN
-F 2 "" H 6700 4800 60  0000 C CNN
+F 2 "REInnovationFootprint:C_1V7_TH" H 6700 4800 60  0001 C CNN
 F 3 "" H 6700 4800 60  0000 C CNN
 	1    6700 4800
-	1    0    0    -1
-$EndComp
-$Comp
-L MCP1703-Matt U4
-U 1 1 5467B677
-P 9550 5100
-F 0 "U4" H 9700 4904 60  0000 C CNN
-F 1 "MCP1826S" H 9550 5300 60  0000 C CNN
-F 2 "~" H 9550 5100 60  0000 C CNN
-F 3 "http://docs-europe.electrocomponents.com/webdocs/137e/0900766b8137eda2.pdf" H 9550 5100 60  0001 C CNN
-F 4 "~" H 9550 5100 60  0000 C CNN "Notes"
-F 5 "1A LDO low Iq" H 9550 5100 60  0001 C CNN "Description"
-F 6 "Microchip" H 9550 5100 60  0001 C CNN "Manufacturer"
-F 7 "MCP1826S-3302E/AB" H 9550 5100 60  0001 C CNN "Manufacturer Part No"
-F 8 "RS" H 9550 5100 60  0001 C CNN "Supplier 1"
-F 9 "669-5174" H 9550 5100 60  0001 C CNN "Supplier 1 Part No"
-F 10 "0.76" H 9550 5100 60  0001 C CNN "Supplier 1 Cost"
-F 11 "~" H 9550 5100 60  0001 C CNN "Supplier 2"
-F 12 "~" H 9550 5100 60  0001 C CNN "Supplier 2 Part No"
-F 13 "~" H 9550 5100 60  0001 C CNN "Supplier 2 Cost"
-	1    9550 5100
 	1    0    0    -1
 $EndComp
@@
 F 0 "U3" H 3200 1250 60  0000 C CNN
 F 1 "LM2574" H 3200 1400 60  0000 C CNN
-F 2 "" H 3200 1200 60  0000 C CNN
-F 3 "" H 3200 1200 60  0000 C CNN
+F 2 "REInnovationFootprint:DIP-8_300_ELL" H 3200 1200 60  0001 C CNN
+F 3 "http://www.ti.com/lit/ds/symlink/lm2574.pdf" H 3200 1200 60  0001 C CNN
+F 4 "~" H 3200 1200 60  0000 C CNN "Notes"
+F 5 "0.5A step down DC-DC" H 3200 1200 60  0001 C CNN "Description"
+F 6 "TI" H 3200 1200 60  0001 C CNN "Manufacturer"
+F 7 "LM2574" H 3200 1200 60  0001 C CNN "Manufacturer Part No"
+F 8 "RS" H 3200 1200 60  0001 C CNN "Supplier 1"
+F 9 "~" H 3200 1200 60  0001 C CNN "Supplier 1 Part No"
+F 10 "~" H 3200 1200 60  0001 C CNN "Supplier 1 Cost"
+F 11 "~" H 3200 1200 60  0001 C CNN "Supplier 2"
+F 12 "~" H 3200 1200 60  0001 C CNN "Supplier 2 Part No"
+F 13 "~" H 3200 1200 60  0001 C CNN "Supplier 2 Cost"
 	1    3200 1200
 	1    0    0    -1
@@
 F 0 "C9" H 2050 1450 50  0000 L CNN
 F 1 "22uF" H 2050 1250 50  0000 L CNN
-F 2 "" H 2000 1350 60  0001 C CNN
+F 2 "REInnovationFootprint:C_1V7_TH" H 2000 1350 60  0001 C CNN
 F 3 "" H 2000 1350 60  0001 C CNN
 F 4 "~" H 2000 1350 60  0001 C CNN "Description"
@@
 F 0 "C12" H 5200 1600 50  0000 L CNN
 F 1 "220uF" H 5200 1400 50  0000 L CNN
-F 2 "" H 5150 1500 60  0001 C CNN
+F 2 "REInnovationFootprint:C_1V7_TH" H 5150 1500 60  0001 C CNN
 F 3 "" H 5150 1500 60  0001 C CNN
 F 4 "~" H 5150 1500 60  0001 C CNN "Description"
@@
 F 0 "L1" V 4600 1200 50  0000 C CNN
 F 1 "330uH" V 4750 1200 50  0000 C CNN
-F 2 "" H 4650 1200 50  0000 C CNN
+F 2 "REInnovationFootprint:TH_Inductor" H 4650 1200 50  0001 C CNN
 F 3 "" H 4650 1200 50  0000 C CNN
 	1    4650 1200
@@
 F 0 "D10" H 4150 1600 50  0000 C CNN
 F 1 "1N5819" H 4150 1400 50  0000 C CNN
-F 2 "" H 4150 1500 50  0000 C CNN
+F 2 "REInnovationFootprint:TH_Diode_1" H 4150 1500 50  0001 C CNN
 F 3 "" H 4150 1500 50  0000 C CNN
 	1    4150 1500
@@
 F 0 "U5" H 5550 4650 60  0000 C CNN
 F 1 "MCP73832" H 5400 5550 60  0000 C CNN
-F 2 "" H 5500 4700 60  0000 C CNN
+F 2 "REInnovationFootprint:SM_SOT-23-5" H 5500 4700 60  0001 C CNN
 F 3 "http://ww1.microchip.com/downloads/en/DeviceDoc/20001984g.pdf" H 5500 4700 60  0001 C CNN
 F 4 "~" H 5500 4700 60  0000 C CNN "Notes"
@@
 F 0 "D11" H 6050 2350 50  0000 C CNN
 F 1 "D_Schottky" H 6050 2150 50  0000 C CNN
-F 2 "" H 6050 2250 50  0000 C CNN
+F 2 "REInnovationFootprint:TH_Diode_1" H 6050 2250 50  0001 C CNN
 F 3 "" H 6050 2250 50  0000 C CNN
 	1    6050 2250
@@
 F 0 "D12" H 6050 2800 50  0000 C CNN
 F 1 "D_Schottky" H 6050 2600 50  0000 C CNN
-F 2 "" H 6050 2700 50  0000 C CNN
+F 2 "REInnovationFootprint:TH_Diode_1" H 6050 2700 50  0001 C CNN
 F 3 "" H 6050 2700 50  0000 C CNN
 	1    6050 2700
@@
 F 0 "Q2" H 9450 2600 50  0000 R CNN
 F 1 "RFU9110PBF" H 9800 2500 50  0000 R CNN
-F 2 "" H 9350 2650 50  0000 C CNN
+F 2 "REInnovationFootprint:TO220_P_FET" H 9350 2650 50  0001 C CNN
 F 3 "http://docs-europe.electrocomponents.com/webdocs/0791/0900766b807912ad.pdf" H 9150 2550 50  0001 C CNN
 F 4 "~" H 9150 2550 60  0000 C CNN "Notes"
@@
 F 0 "D14" H 9700 2500 50  0000 C CNN
 F 1 "D_Schottky" H 9700 2300 50  0000 C CNN
-F 2 "" H 9700 2400 50  0000 C CNN
+F 2 "REInnovationFootprint:TH_Diode_1" H 9700 2400 50  0001 C CNN
 F 3 "" H 9700 2400 50  0000 C CNN
 	1    9700 2400
@@
 F 0 "R18" V 8680 2200 50  0000 C CNN
 F 1 "100k" V 8600 2200 50  0000 C CNN
-F 2 "" V 8530 2200 50  0000 C CNN
+F 2 "REInnovationFootprint:TH_Resistor_1" V 8530 2200 50  0001 C CNN
 F 3 "" H 8600 2200 50  0000 C CNN
 	1    8600 2200
@@
 AR Path="/546244C7/57A0C9C8" Ref="D13"  Part="1"
 F 0 "D13" H 6050 4850 50  0000 C CNN
-F 1 "LED" H 6050 4650 50  0000 C CNN
-F 2 "" H 6050 4750 50  0000 C CNN
+F 1 "CHRG" H 6050 4650 50  0000 C CNN
+F 2 "REInnovationFootprint:TH_LED-5MM_larg_pad" H 6050 4750 50  0001 C CNN
 F 3 "" H 6050 4750 50  0000 C CNN
 	1    6050 4750
@@
 F 0 "SW3" H 10550 3450 50  0000 C CNN
 F 1 "ON/OFF" H 10550 3250 50  0000 C CNN
-F 2 "" H 10550 3350 50  0000 C CNN
+F 2 "matts_components:SW_SPDT_rapid_760271" H 10550 3350 50  0001 C CNN
 F 3 "" H 10550 3350 50  0000 C CNN
 	1    10550 3350
@@
 F 0 "D18" H 6050 3150 50  0000 C CNN
 F 1 "D_Schottky" H 6050 2950 50  0000 C CNN
-F 2 "" H 6050 3050 50  0000 C CNN
+F 2 "REInnovationFootprint:TH_Diode_1" H 6050 3050 50  0001 C CNN
 F 3 "" H 6050 3050 50  0000 C CNN
 	1    6050 3050
@@
 Wire Wire Line
 	8150 5050 9150 5050
+$Comp
+L MCP1826S U2
+U 1 1 58F214B0
+P 9550 5100
+F 0 "U2" H 9700 4904 60  0000 C CNN
+F 1 "MCP1826S" H 9550 5300 60  0000 C CNN
+F 2 "REInnovationFootprint:TO220_MCP1826S" H 9550 5100 60  0001 C CNN
+F 3 "" H 9550 5100 60  0000 C CNN
+	1    9550 5100
+	1    0    0    -1
+$EndComp
 $EndSCHEMATC

Commit message: BOM uploaded
Parts:
- SW3: symbol SPST -> SPST-RESCUE-RELogger_PCB_v1
- U2: symbol MCP1826S -> MCP1826S-RESCUE-RELogger_PCB_v1
Connections:
- net Vss: no longer SW3.2
- net at D14.1 (K), Q2.3 (S): no longer SW3.1
Changed lines of the file:
@@
 LIBS:matts_components
 LIBS:linear2
+LIBS:ds3231
+LIBS:micro_sd
 LIBS:RELogger_PCB_v1-cache
 EELAYER 25 0
@@
 Connection ~ 7200 3050
 $Comp
-L SPST SW3
+L SPST-RESCUE-RELogger_PCB_v1 SW3
 U 1 1 57B5BF9D
 P 10550 3350
@@
 	8150 5050 9150 5050
 $Comp
-L MCP1826S U2
+L MCP1826S-RESCUE-RELogger_PCB_v1 U2
 U 1 1 58F214B0
 P 9550 5100

Commit message: Re load of new PCB
Parts:
- SW3: symbol SPST-RESCUE-RELogger_PCB_v1 -> SPST
- U2: symbol MCP1826S-RESCUE-RELogger_PCB_v1 -> MCP1826S
Connections:
- net Vss: now also SW3.2
- net at D14.1 (K), Q2.3 (S): now also SW3.1
Changed lines of the file:
@@
 LIBS:matts_components
 LIBS:linear2
-LIBS:ds3231
-LIBS:micro_sd
 LIBS:RELogger_PCB_v1-cache
 EELAYER 25 0
@@
 Connection ~ 7200 3050
 $Comp
-L SPST-RESCUE-RELogger_PCB_v1 SW3
+L SPST SW3
 U 1 1 57B5BF9D
 P 10550 3350
@@
 	8150 5050 9150 5050
 $Comp
-L MCP1826S-RESCUE-RELogger_PCB_v1 U2
+L MCP1826S U2
 U 1 1 58F214B0
 P 9550 5100
